Commit message: Gazebo plugins added for control the tinybot

File: tinybot_ws/src/tinybot_description/urdf/mobile_base.xacro (robot description, xacro)
@@ -24,5 +24,5 @@
                        h="${2*base_height}" xyz="0 0 ${base_height / 2.0}" rpy="0 0 0"/>
   </link>
-  <xacro:macro name="wheel_link" params="prefix">
+  <xacro:macro name="Wheel_link" params="prefix">
     <link name="${prefix}Wheel_link">
       <visual>
@@ -43,6 +43,6 @@
     </link>
   </xacro:macro>
-  <xacro:wheel_link prefix="right"/>
-  <xacro:wheel_link prefix="left"/>
+  <xacro:Wheel_link prefix="right"/>
+  <xacro:Wheel_link prefix="left"/>
   <link name="casterWheel">
     <visual>

File: tinybot_ws/src/tinybot_description/urdf/mobile_base_gazebo.xacro (robot description, xacro)
@@ -4,12 +4,31 @@
         <material>Gazebo/Blue</material>
     </gazebo>
-    <gazebo reference="rightwheel_link">
+    <gazebo reference="rightWheel_link">
         <material>Gazebo/White</material>
     </gazebo>
-    <gazebo reference="lefttwheel_link">
+    <gazebo reference="leftWheel_link">
         <material>Gazebo/White</material>
     </gazebo>
-    <gazebo reference="casterwheel_link">
+    <gazebo reference="casterWheel">
         <material>Gazebo/White</material>
     </gazebo>
+    <gazebo>
+        <plugin name="diff_drive_controller" filename="libgazebo_ros_diff_drive.so">
+            <!-- Update rate in Hz -->
+            <update_rate>50</update_rate>
+            <!-- wheels -->
+            <left_joint>base_leftWheel_joint</left_joint>
+            <right_joint>base_rightWheel_joint</right_joint>
+            <!-- kinematics -->
+            <wheel_separation>0.45</wheel_separation>
+            <wheel_diameter>0.2</wheel_diameter>
+            <!-- output -->
+            <publish_odom>true</publish_odom>
+            <publish_odom_tf>true</publish_odom_tf>
+            <publish_wheel_tf>true</publish_wheel_tf>
+            <odometry_topic>odom</odometry_topic>
+            <odometry_frame>odom</odometry_frame>
+            <robot_base_frame>base_footprint</robot_base_frame>
+        </plugin>
+    </gazebo>
 </robot>
